Commit message: elsa_simulator package created which uses original packages to build elsa specific simulator (seperate perception launch and urdf with camera)

File: elsa_simulator/robots/_d435.urdf.xacro (robot description, xacro)
@@ -8,5 +8,5 @@
 <robot name="sensor_d435" xmlns:xacro="http://ros.org/wiki/xacro">
   <!--File includes-->
-  <xacro:include filename="$(find realsense2_description)/urdf/_d435.gazebo.xacro"/>
+  <xacro:include filename="$(find elsa_simulator)/robots/_d435.gazebo.xacro"/>
   <xacro:macro name="sensor_d435" params="name:=camera topics_ns:=camera parent *origin publish_pointcloud:=true">
     <xacro:property name="M_PI" value="3.1415926535897931" />

File: franka_panda_description/robots/panda_arm_hand.urdf.xacro (robot description, xacro)
@@ -7,22 +7,4 @@
   <xacro:arg name="connected_to" default=""/> <!-- If using a different frame with ${connected_to} param, make sure 'world' frame exists in the TF tree -->
   <xacro:include filename="$(find franka_panda_description)/robots/panda_arm.xacro"/>
-  <!-- Real Sense Camera -->
-  <xacro:include filename="$(find franka_panda_description)/robots/_d435.urdf.xacro" />
-  <link name="camera_base">
-    <!-- <visual>
-      <origin xyz="0.4 0 1.5" rpy="0 1.57 0" />
-      <geometry>
-        <box size="0.03 0.05 0.03" />
-      </geometry>
-    </visual> -->
-  </link>
-  <joint name="cam_joint" type="fixed">
-    <parent link="panda_link0"/>
-    <child link="camera_base"/>
-  </joint>
-  <xacro:sensor_d435 name="camera" topics_ns="camera" parent="camera_base" publish_pointcloud="true">
-    <origin xyz="0.5 0 1" rpy="0 1.57 0" />
-  </xacro:sensor_d435>
-  <!-- Real Sense Camera End -->
   <xacro:if value="$(arg load_gripper)">
     <xacro:include filename="$(find franka_panda_description)/robots/hand.xacro"/>
