Commit message: Added robot_body_filter submodule

File: franka_panda_description/robots/hand.xacro (robot description, xacro)
@@ -13,5 +13,5 @@
     </xacro:unless>
     <link name="${ns}_hand">
-      <visual>
+      <!-- <visual>
         <geometry>
           <mesh filename="package://franka_panda_description/meshes/visual/hand.dae"/>
@@ -22,5 +22,5 @@
           <mesh filename="package://franka_panda_description/meshes/collision/hand.stl"/>
         </geometry>
-      </collision>
+      </collision> -->
       <inertial>
         <origin rpy="0 0 0" xyz="0 0.0015244 0.0275912"/>
@@ -30,5 +30,5 @@
     </link>
     <link name="${ns}_leftfinger">
-      <visual>
+      <!-- <visual>
         <geometry>
           <mesh filename="package://franka_panda_description/meshes/visual/finger.dae"/>
@@ -39,5 +39,5 @@
           <mesh filename="package://franka_panda_description/meshes/collision/finger.stl"/>
         </geometry>
-      </collision>
+      </collision> -->
       <inertial>
         <origin rpy="0 0 0" xyz="0 0.0145644 0.0227941"/>
@@ -47,5 +47,5 @@
     </link>
     <link name="${ns}_rightfinger">
-      <visual>
+      <!-- <visual>
         <origin xyz="0 0 0" rpy="0 0 ${pi}"/>
         <geometry>
@@ -58,5 +58,5 @@
           <mesh filename="package://franka_panda_description/meshes/collision/finger.stl"/>
         </geometry>
-      </collision>
+      </collision> -->
       <inertial>
         <origin rpy="0 0 3.141592653589793" xyz="0 -0.0145644 0.0227941"/>

File: franka_panda_description/robots/panda_arm.xacro (robot description, xacro)
@@ -145,5 +145,5 @@
     </joint>
     <link name="${arm_id}_link5">
-      <visual>
+      <!-- <visual>
         <geometry>
           <mesh filename="package://${description_pkg}/meshes/visual/link5.dae"/>
@@ -154,5 +154,5 @@
           <mesh filename="package://${description_pkg}/meshes/collision/link5.stl"/>
         </geometry>
-      </collision>
+      </collision> -->
       <inertial>
         <origin xyz="-1.1953e-02 4.1065e-02 -3.8437e-02" rpy="0 0 0"/>
@@ -177,7 +177,11 @@
       </visual>
       <collision>
-        <geometry>
+        <!-- <geometry>
           <mesh filename="package://${description_pkg}/meshes/collision/link6.stl"/>
-        </geometry>
+        </geometry> -->
+         <geometry>
+          <box size="0.1 0.07 0.06"/>
+        </geometry>
+        <origin rpy="0 0 0" xyz="0.04 0.01 0.0"/>
       </collision>
       <inertial>
@@ -197,5 +201,5 @@
     </joint>
     <link name="${arm_id}_link7">
-      <visual>
+      <!-- <visual>
         <geometry>
           <mesh filename="package://${description_pkg}/meshes/visual/link7.dae"/>
@@ -206,5 +210,5 @@
           <mesh filename="package://${description_pkg}/meshes/collision/link7.stl"/>
         </geometry>
-      </collision>
+      </collision> -->
       <inertial>
         <origin xyz="1.0517e-02 -4.252e-03 6.1597e-02" rpy="0 0 0"/>
